Commit message: fix rotation error & wheels axis

File: ros2_ws/src/ugv_gazebo_sim/scout/scout_description/urdf/scout_mini.xacro (robot description, xacro)
@@ -1,5 +1,19 @@
 <?xml version="1.0"?>
 <robot name="scout_mini" xmlns:xacro="http://ros.org/wiki/xacro">
-    <!-- Vehicle Geometries -->
+    <!-- ==== Wheel parameters (from manual & Meshlab) ==== -->
+    <!-- 타이어 지름 ≈ 0.16m → 반지름 0.08m -->
+    <xacro:property name="wheel_radius" value="0.08"/>
+    <!-- Meshlab Bounding Box 두께 ≈ 0.132m -->
+    <xacro:property name="wheel_length" value="0.08"/>
+    <!-- ================= Vehicle Geometries ================= -->
+    <!-- 바닥 기준 프레임 -->
+    <link name="base_footprint" />
+    <!-- base_footprint -> base_link 고정 변환 -->
+    <joint name="base_footprint_to_base_link" type="fixed">
+        <!-- 휠 중심이 지면에서 0.08m가 되도록: z = 0.18m (휠 중심 z = -0.10m) -->
+        <origin xyz="0 0 0.18" rpy="0 0 0" />
+        <parent link="base_footprint" />
+        <child link="base_link" />
+    </joint>
     <!-- Base link -->
     <link name="base_link">
@@ -7,140 +21,244 @@
             <origin xyz="0 0 0" rpy="1.57 0 -1.57" />
             <geometry>
-                <mesh
-                    filename="package://scout_description/meshes/scout_mini_base_link.dae" />
-            </geometry>
-        </visual>
-        <collision>
-            <origin xyz="0 0 0" rpy="1.57 0 -1.57" />
-            <geometry>
-                <mesh
-                    filename="package://scout_description/meshes/scout_mini_base_link.dae" />
-            </geometry>
-        </collision>
-    </link>
-    <link
-        name="inertial_link">
-        <inertial>
-            <mass value="132.3898489950015" />
-            <origin xyz=" 0 0 0" />
-            <inertia ixx="0.185196122711036" ixy="4.30144213829512E-08" ixz="5.81037523686401E-08"
-                iyy="0.364893736238929" iyz="-0.000386720198091934" izz="0.223868521722778" />
-        </inertial>
-    </link>
-    <joint
-        name="inertial_joint" type="fixed">
+                <mesh filename="package://scout_description/meshes/mini_body.dae" />
+            </geometry>
+        </visual>
+        <!-- Meshlab 기준 scout_mini_base_link.dae Bounding Box
+             Size: 0.389876 0.182181 0.560607 (X Y Z)
+             -> 동일 축 기준 box collision으로 근사 -->
+        <collision>
+            <origin xyz="0 0 -0.0215" rpy="1.57 0 -1.57" />
+            <geometry>
+                <box size="0.389876 0.182181 0.560607" />
+            </geometry>
+        </collision>
+    </link>
+    <!-- 차체 관성 링크 (총 질량 23kg 중 19kg) -->
+    <link name="inertial_link">
+        <inertial>
+            <mass value="19.0" />
+            <!-- 질량중심을 base_link 원점과 일치시킴 -->
+            <origin xyz="0 0 0" />
+            <!-- 0.612 x 0.580 x 0.245 m, m=19kg 직육면체 근사 관성 -->
+            <inertia
+                ixx="0.627673"
+                ixy="0.0"
+                ixz="0.0"
+                iyy="0.688068"
+                iyz="0.0"
+                izz="1.125661" />
+        </inertial>
+    </link>
+    <joint name="inertial_joint" type="fixed">
         <origin xyz="0 0 0" rpy="0 0 0" />
         <parent link="base_link" />
         <child link="inertial_link" />
     </joint>
-    <!-- Scout wheel -->
-    <link
-        name="front_right_wheel_link">
-        <inertial>
-            <mass value="3" />
-            <origin xyz="0 0 0" />
-            <inertia ixx="0.7171" ixy="0" ixz="0" iyy="0.7171" iyz="0" izz="0.1361" />
-        </inertial>
-        <visual>
-            <origin xyz="0 0 0" rpy="0 0 0" />
-            <geometry>
-                <mesh filename="package://scout_description/meshes/wheel.dae" />
-            </geometry>
-        </visual>
-        <collision>
-            <origin xyz="0 0 0" rpy="0 0 0" />
-            <geometry>
-                <mesh filename="package://scout_description/meshes/wheel.dae" />
-            </geometry>
-        </collision>
-    </link>
-    <joint
-        name="front_right_wheel" type="continuous">
-        <origin rpy="1.57 0 0" xyz="0.2319755 -0.2082515 -0.099998" />
+    <!-- ======================= Scout wheels ======================= -->
+    <!-- Meshlab 기준 wheel.dae Bounding Box:
+         Size: 0.159896 0.159953 0.132000
+         -> 지름 ≈ 0.16m (반지름 ≈ 0.08m), 두께 ≈ 0.132m
+         -> cylinder(radius=wheel_radius, length=wheel_length)로 근사 -->
+    <!-- Front Right Wheel -->
+    <link name="front_right_wheel_link">
+        <inertial>
+            <mass value="1.0" />
+            <origin xyz="0 0 0" />
+            <inertia
+                ixx="0.002013"
+                ixy="0.0"
+                ixz="0.0"
+                iyy="0.002013"
+                iyz="0.0"
+                izz="0.002685" />
+        </inertial>
+        <visual>
+            <origin xyz="0 -0.0375 0" rpy="0 0 0" />
+            <geometry>
+                <mesh filename="package://scout_description/meshes/right_wheel_mini_2.dae" />
+            </geometry>
+        </visual>
+        <collision>
+            <!-- 좌우 방향으로 1.5cm 바깥으로 이동 (joint의 Rx 때문에 base y로 투영됨) -->
+            <origin xyz="0 -0.04 0" rpy="1.57 0 0" />
+            <geometry>
+                <cylinder length="${wheel_length}" radius="${wheel_radius}" />
+            </geometry>
+            <!-- v2와 동일 패턴의 contact / friction 설정 -->
+            <surface>
+                <contact>
+                    <ode>
+                        <min_depth>0.001</min_depth>
+                        <kp>1000000000.0</kp>
+                        <kd>0.0</kd>
+                    </ode>
+                </contact>
+                <friction>
+                    <ode>
+                        <mu>0.9</mu>
+                        <mu2>0.7</mu2>
+                        <fdir1>1 0 0</fdir1>
+                    </ode>
+                </friction>
+            </surface>
+        </collision>
+    </link>
+    <joint name="front_right_wheel" type="continuous">
+        <!-- 축 기준 트랙폭 0.420m → y = ±0.205 -->
+        <origin xyz="0.2255 -0.205 -0.10" rpy="0 0 0" />
         <parent link="base_link" />
         <child link="front_right_wheel_link" />
-        <axis xyz="0 0 -1" rpy="0 0 0" />
-    </joint>
+        <!-- 회전축: link z축(바퀴 회전) -->
+        <axis xyz="0 1 0" rpy="0 0 0" />
+    </joint>
+    <!-- Front Left Wheel -->
     <link name="front_left_wheel_link">
         <inertial>
-            <mass value="3" />
-            <origin xyz="0 0 0" />
-            <inertia ixx="0.7171" ixy="0" ixz="0" iyy="0.7171" iyz="0" izz="0.1361" />
-        </inertial>
-        <visual>
-            <origin xyz="0 0 0" rpy="0 0 0" />
-            <geometry>
-                <mesh filename="package://scout_description/meshes/wheel.dae" />
-            </geometry>
-        </visual>
-        <collision>
-            <origin xyz="0 0 0" rpy="0 0 0" />
-            <geometry>
-                <mesh filename="package://scout_description/meshes/wheel.dae" />
-            </geometry>
-        </collision>
-    </link>
-    <joint
-        name="front_left_wheel" type="continuous">
-        <origin rpy="-1.57 0 0" xyz="0.2319755 0.2082515 -0.100998" />
+            <mass value="1.0" />
+            <origin xyz="0 0 0" />
+            <inertia
+                ixx="0.002013"
+                ixy="0.0"
+                ixz="0.0"
+                iyy="0.002013"
+                iyz="0.0"
+                izz="0.002685" />
+        </inertial>
+        <visual>
+            <origin xyz="0 0.0375 0" rpy="0 0 0" />
+            <geometry>
+                <mesh filename="package://scout_description/meshes/left_wheel_mini_2.dae" />
+            </geometry>
+        </visual>
+        <collision>
+            <origin xyz="0 0.04 0" rpy="-1.57 0 0" />
+            <geometry>
+                <cylinder length="${wheel_length}" radius="${wheel_radius}" />
+            </geometry>
+            <surface>
+                <contact>
+                    <ode>
+                        <min_depth>0.001</min_depth>
+                        <kp>1000000000.0</kp>
+                        <kd>0.0</kd>
+                    </ode>
+                </contact>
+                <friction>
+                    <ode>
+                        <mu>0.9</mu>
+                        <mu2>0.7</mu2>
+                        <fdir1>1 0 0</fdir1>
+                    </ode>
+                </friction>
+            </surface>
+        </collision>
+    </link>
+    <joint name="front_left_wheel" type="continuous">
+        <origin xyz="0.2255 0.205 -0.10" rpy="0 0 0" />
         <parent link="base_link" />
         <child link="front_left_wheel_link" />
-        <axis xyz="0 0 1" rpy="0 0 0" />
-    </joint>
+        <axis xyz="0 1 0" rpy="0 0 0" />
+    </joint>
+    <!-- Rear Right Wheel -->
     <link name="rear_right_wheel_link">
         <inertial>
-            <mass value="3" />
-            <origin xyz="0 0 0" />
-            <inertia ixx="0.7171" ixy="0" ixz="0" iyy="0.7171" iyz="0" izz="0.1361" />
-        </inertial>
-        <visual>
-            <origin xyz="0 0 0" rpy="0 0 0" />
-            <geometry>
-                <mesh filename="package://scout_description/meshes/wheel.dae" />
-            </geometry>
-        </visual>
-        <collision>
-            <origin xyz="0 0 0" rpy="0 0 0" />
-            <geometry>
-                <mesh filename="package://scout_description/meshes/wheel.dae" />
-            </geometry>
-        </collision>
-    </link>
-    <joint
-        name="rear_right_wheel" type="continuous">
-        <origin rpy="1.57 0 0" xyz="-0.2319755 -0.2082515 -0.099998" />
+            <mass value="1.0" />
+            <origin xyz="0 0 0" />
+            <inertia
+                ixx="0.002013"
+                ixy="0.0"
+                ixz="0.0"
+                iyy="0.002013"
+                iyz="0.0"
+                izz="0.002685" />
+        </inertial>
+        <visual>
+            <origin xyz="0 -0.0375 0" rpy="0 0 0" />
+            <geometry>
+                <mesh filename="package://scout_description/meshes/right_wheel_mini_2.dae" />
+            </geometry>
+        </visual>
+        <collision>
+            <origin xyz="0 -0.04 0" rpy="1.57 0 0" />
+            <geometry>
+                <cylinder length="${wheel_length}" radius="${wheel_radius}" />
+            </geometry>
+            <surface>
+                <contact>
+                    <ode>
+                        <min_depth>0.001</min_depth>
+                        <kp>1000000000.0</kp>
+                        <kd>0.0</kd>
+                    </ode>
+                </contact>
+                <friction>
+                    <ode>
+                        <mu>0.9</mu>
+                        <mu2>0.7</mu2>
+                        <fdir1>1 0 0</fdir1>
+                    </ode>
+                </friction>
+            </surface>
+        </collision>
+    </link>
+    <joint name="rear_right_wheel" type="continuous">
+        <origin xyz="-0.2255 -0.205 -0.10" rpy="0 0 0" />
         <parent link="base_link" />
         <child link="rear_right_wheel_link" />
-        <axis xyz="0 0 -1" rpy="0 0 0" />
-    </joint>
+        <axis xyz="0 1 0" rpy="0 0 0" />
+    </joint>
+    <!-- Rear Left Wheel -->
     <link name="rear_left_wheel_link">
         <inertial>
-            <mass value="3" />
-            <origin xyz="0 0 0" />
-            <inertia ixx="0.7171" ixy="0" ixz="0" iyy="0.7171" iyz="0" izz="0.1361" />
-        </inertial>
-        <visual>
-            <origin xyz="0 0 0" rpy="0 0 0" />
-            <geometry>
-                <mesh filename="package://scout_description/meshes/wheel.dae" />
-            </geometry>
-        </visual>
-        <collision>
-            <origin xyz="0 0 0" rpy="0 0 0" />
-            <geometry>
-                <mesh filename="package://scout_description/meshes/wheel.dae" />
-            </geometry>
-        </collision>
-    </link>
-    <joint
-        name="rear_left_wheel" type="continuous">
-        <origin rpy="-1.57 0 0" xyz="-0.2319755 0.2082515 -0.100998" />
+            <mass value="1.0" />
+            <origin xyz="0 0 0" />
+            <inertia
+                ixx="0.002013"
+                ixy="0.0"
+                ixz="0.0"
+                iyy="0.002013"
+                iyz="0.0"
+                izz="0.002685" />
+        </inertial>
+        <visual>
+            <origin xyz="0 0.0375 0" rpy="0 0 0" />
+            <geometry>
+                <mesh filename="package://scout_description/meshes/left_wheel_mini_2.dae" />
+            </geometry>
+        </visual>
+        <collision>
+            <origin xyz="0 0.04 0" rpy="-1.57 0 0" />
+            <geometry>
+                <cylinder length="${wheel_length}" radius="${wheel_radius}" />
+            </geometry>
+            <surface>
+                <contact>
+                    <ode>
+                        <min_depth>0.001</min_depth>
+                        <kp>1000000000.0</kp>
+                        <kd>0.0</kd>
+                    </ode>
+                </contact>
+                <friction>
+                    <ode>
+                        <mu>0.9</mu>
+                        <mu2>0.7</mu2>
+                        <fdir1>1 0 0</fdir1>
+                    </ode>
+                </friction>
+            </surface>
+        </collision>
+    </link>
+    <joint name="rear_left_wheel" type="continuous">
+        <origin xyz="-0.2255 0.205 -0.10" rpy="0 0 0" />
         <parent link="base_link" />
         <child link="rear_left_wheel_link" />
-        <axis xyz="0 0 1" rpy="0 0 0" />
-    </joint>
-    <!-- Scout gazebo plugin -->
+        <axis xyz="0 1 0" rpy="0 0 0" />
+    </joint>
+    <!-- ===================== Scout gazebo plugin ===================== -->
     <gazebo>
-        <plugin filename="libignition-gazebo-joint-state-publisher-system.so"
+        <!-- Joint states -->
+        <plugin
+            filename="libignition-gazebo-joint-state-publisher-system.so"
             name="ignition::gazebo::systems::JointStatePublisher">
             <topic>joint_states</topic>
@@ -151,23 +269,39 @@
             <joint_name>rear_left_wheel</joint_name>
         </plugin>
+        <!-- Skid-steer DiffDrive -->
         <plugin
             filename="libignition-gazebo-diff-drive-system.so"
             name="ignition::gazebo::systems::DiffDrive">
             <left_joint>front_left_wheel</left_joint>
+            <left_joint>rear_left_wheel</left_joint>
             <right_joint>front_right_wheel</right_joint>
-            <left_joint>rear_left_wheel</left_joint>
             <right_joint>rear_right_wheel</right_joint>
-            <wheel_separation>0.490</wheel_separation>
-            <wheel_radius>0.160</wheel_radius>
-            <!-- limits -->
-            <max_wheel_torque>20</max_wheel_torque>
-            <max_linear_acceleration>1.0</max_linear_acceleration>
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
Commit message: Fix: Absorb hospital world package into main repo

File: ros2_ws/src/ugv_gazebo_sim/scout/scout_description/urdf/scout_mini.xacro (robot description, xacro)
@@ -63,13 +63,14 @@
     <link name="front_right_wheel_link">
         <inertial>
-            <mass value="1.0" />
-            <origin xyz="0 0 0" />
-            <inertia
-                ixx="0.002013"
-                ixy="0.0"
-                ixz="0.0"
-                iyy="0.002013"
-                iyz="0.0"
-                izz="0.002685" />
+            <!-- 질량/관성 상향 (기존 1.0 / 0.002013 등에서 4배 증가) -->
+            <mass value="4.0" />
+            <origin xyz="0 0 0" />
+            <inertia
+                ixx="0.008052"
+                ixy="0.0"
+                ixz="0.0"
+                iyy="0.008052"
+                iyz="0.0"
+                izz="0.010740" />
         </inertial>
         <visual>
@@ -111,17 +112,19 @@
         <!-- 회전축: link z축(바퀴 회전) -->
         <axis xyz="0 1 0" rpy="0 0 0" />
+        <!-- 조인트 마찰 완화 (20 -> 4) -->
+        <dynamics damping="0.0" friction="4.0" />
     </joint>
     <!-- Front Left Wheel -->
     <link name="front_left_wheel_link">
         <inertial>
-            <mass value="1.0" />
-            <origin xyz="0 0 0" />
-            <inertia
-                ixx="0.002013"
-                ixy="0.0"
-                ixz="0.0"
-                iyy="0.002013"
-                iyz="0.0"
-                izz="0.002685" />
+            <mass value="4.0" />
+            <origin xyz="0 0 0" />
+            <inertia
+                ixx="0.008052"
+                ixy="0.0"
+                ixz="0.0"
+                iyy="0.008052"
+                iyz="0.0"
+                izz="0.010740" />
         </inertial>
         <visual>
@@ -159,17 +162,18 @@
         <child link="front_left_wheel_link" />
         <axis xyz="0 1 0" rpy="0 0 0" />
+        <dynamics damping="0.0" friction="4.0" />
     </joint>
     <!-- Rear Right Wheel -->
     <link name="rear_right_wheel_link">
         <inertial>
-            <mass value="1.0" />
-            <origin xyz="0 0 0" />
-            <inertia
-                ixx="0.002013"
-                ixy="0.0"
-                ixz="0.0"
-                iyy="0.002013"
-                iyz="0.0"
-                izz="0.002685" />
+            <mass value="4.0" />
+            <origin xyz="0 0 0" />
+            <inertia
+                ixx="0.008052"
+                ixy="0.0"
+                ixz="0.0"
+                iyy="0.008052"
+                iyz="0.0"
+                izz="0.010740" />
         </inertial>
         <visual>
@@ -207,17 +211,18 @@
         <child link="rear_right_wheel_link" />
         <axis xyz="0 1 0" rpy="0 0 0" />
+        <dynamics damping="0.0" friction="4.0" />
     </joint>
     <!-- Rear Left Wheel -->
     <link name="rear_left_wheel_link">
         <inertial>
-            <mass value="1.0" />
-            <origin xyz="0 0 0" />
-            <inertia
-                ixx="0.002013"
-                ixy="0.0"
-                ixz="0.0"
-                iyy="0.002013"
-                iyz="0.0"
-                izz="0.002685" />
+            <mass value="4.0" />
+            <origin xyz="0 0 0" />
+            <inertia
+                ixx="0.008052"
+                ixy="0.0"
+                ixz="0.0"
+                iyy="0.008052"
+                iyz="0.0"
+                izz="0.010740" />
         </inertial>
         <visual>
@@ -255,4 +260,5 @@
         <child link="rear_left_wheel_link" />
         <axis xyz="0 1 0" rpy="0 0 0" />
+        <dynamics damping="0.0" friction="4.0" />
     </joint>
     <!-- ===================== Scout gazebo plugin ===================== -->
@@ -278,5 +284,6 @@
             <right_joint>rear_right_wheel</right_joint>
             <!-- 메뉴얼 기준 접지 기준 트랙폭 0.490m / 모델 축 간격 0.420m -->
-            <wheel_separation>0.410</wheel_separation>
+            <!-- 실제 축 간격(±0.205)을 반영하여 0.410으로 수정 -->
+            <wheel_separation>0.490</wheel_separation>
             <wheel_radius>0.080</wheel_radius>
             <!-- torque는 그대로 두고, 속도/가속도 제한을 설정 -->
@@ -284,10 +291,12 @@
             <max_linear_acceleration>2.0</max_linear_acceleration>
             <min_linear_acceleration>-2.0</min_linear_acceleration>
-            <max_angular_acceleration>5.0</max_angular_acceleration>
-            <min_angular_acceleration>-5.0</min_angular_acceleration>
+            <!-- 각가속도 한계 완화 (±2.0 -> ±1.0) -->
+            <max_angular_acceleration>1.0</max_angular_acceleration>
+            <min_angular_acceleration>-1.0</min_angular_acceleration>
             <max_linear_velocity>10.0</max_linear_velocity>
             <min_linear_velocity>-10.0</min_linear_velocity>
-            <max_angular_velocity>3.0</max_angular_velocity>
-            <min_angular_velocity>-3.0</min_angular_velocity>
+            <!-- 각속도 한계 완화 (±2.0 -> ±1.0) -->
+            <max_angular_velocity>1.0</max_angular_velocity>
+            <min_angular_velocity>-1.0</min_angular_velocity>
             <topic>cmd_vel</topic>
             <!-- 여기서 odom / tf / frame_id / child_frame_id는 제거 -->
