Commit message: fix rglvisualize

File: ros2_ws/src/ouster_simulation/ouster_description/urdf/os1_64.urdf.xacro (robot description, xacro)
@@ -32,8 +32,9 @@
     </link>
     <link name="${name}_lidar">
-      <pose>0 0 0 0 0 ${PI}</pose>
+      <!-- <pose>0 0 0 0 0 ${PI}</pose> -->
     </link>
     <joint name="${name}_lidar_joint" type="fixed">
-      <origin xyz="0 0 0" rpy="0 0 ${PI}" />
+      <!-- <origin xyz="0 0 0" rpy="0 0 ${PI}" /> -->
+      <origin xyz="0 0 0" rpy="0 0 0" />
       <parent link="${name}_sensor"/>
       <child link="${name}_lidar"/>
@@ -59,17 +60,6 @@
           <!-- frame_id in PointCloudPacked header -->
           <frame>${name}_lidar</frame>
-          <!-- Use uniform pattern (no env var required) -->
-          <pattern_uniform>
-            <horizontal>
-              <samples>${samples}</samples>
-              <min_angle>-3.14159</min_angle>
-              <max_angle>3.14159</max_angle>
-            </horizontal>
-            <vertical>
-              <samples>64</samples>
-              <min_angle>${min_angle_v*PI/180.0}</min_angle>
-              <max_angle>${max_angle_v*PI/180.0}</max_angle>
-            </vertical>
-          </pattern_uniform>
+          <!-- Use preset pattern (requires RGL_PATTERNS_DIR env var) -->
+          <pattern_preset>OS1 64</pattern_preset>
         </plugin>
       </sensor>

Commit message: init hunter se robot

File: ros2_ws/src/ouster_simulation/ouster_description/urdf/os1_64.urdf.xacro (robot description, xacro)
@@ -25,5 +25,5 @@
       </collision>
       <visual name="lidar_visual">
-        <origin xyz="0 0 0.3" rpy="0 0 0"/>
+        <origin xyz="0 0 0" rpy="0 0 0"/>
         <geometry>
           <mesh filename="file://$(find ouster_description)/meshes/${file_visual}.dae" />
@@ -57,9 +57,30 @@
           <update_on_paused_sim>false</update_on_paused_sim>
           <!-- Match ros_gz_bridge mapping in your launch -->
-          <topic>/ouster/pointcloud/points</topic>
+          <topic>/scout/pointcloud/points</topic>
           <!-- frame_id in PointCloudPacked header -->
           <frame>${name}_lidar</frame>
-          <!-- Use preset pattern (requires RGL_PATTERNS_DIR env var) -->
-          <pattern_preset>OS1 64</pattern_preset>
+          <!-- Use uniform pattern with explicit vertical FOV -->
+          <!-- NOTE: pattern_preset "OS1 64" has 0° vertical FOV (bug), using pattern_uniform instead -->
+          <!-- Ouster OS1-64: 64 channels, 1024 horizontal samples, ±16.6° vertical FOV -->
+          <!-- Angles in radians: 16.6° = 0.2897 rad, 180° = 3.14159 rad -->
+          <pattern_uniform>
+            <horizontal>
+              <samples>1024</samples>
+              <min_angle>-3.14159</min_angle>
+              <max_angle>3.14159</max_angle>
+            </horizontal>
+            <vertical>
+              <samples>64</samples>
+              <min_angle>-0.2897</min_angle>
+              <max_angle>0.2897</max_angle>
+            </vertical>
+          </pattern_uniform>
+          <!-- Channel configuration for ring ID and timestamp support -->
+          <channels>64</channels>
+          <horizontal_samples>1024</horizontal_samples>
+          <noise>
+            <mean>0.0</mean>
+            <stddev>0.01</stddev>
+          </noise>
         </plugin>
       </sensor>

File: ros2_ws/src/scout_nav2/agilex_scout/urdf/mobile_robot/scout_v2.urdf.xacro (robot description, xacro)
@@ -66,4 +66,17 @@
 		<xacro:include filename="$(find agilex_scout)/urdf/mobile_robot/scout_wheel_type1.xacro" />
 		<xacro:include filename="$(find agilex_scout)/urdf/mobile_robot/scout_wheel_type2.xacro" />
+		<!-- Ouster OS1-64 LiDAR -->
+		<xacro:include filename="$(find ouster_description)/urdf/os1_64.urdf.xacro"/>
+		<xacro:os1_64 parent="mobile_robot_base"
+					  name="os"
+					  hz="10"
+					  samples="1024"
+					  min_range="0.5"
+					  max_range="100.0"
+					  min_angle_v="-21.2"
+					  max_angle_v="21.2"
+					  noise="0.01">
+			<origin xyz="0 0 0.5" rpy="0 0 0"/>
+		</xacro:os1_64>
 		<!-- wheel labeled from 0 to 3, conter-clockwise, starting from front right wheel -->
 		<!-- motor 1 and 2 (left side) are mechanically installed in a reversed direction -->
@@ -82,4 +95,33 @@
 			<child link="front_mount" />
 		</joint>
+		<!-- Intel RealSense D455 RGBD Camera on front_mount -->
+		<xacro:property name="PI" value="3.14159265"/>
+		<joint name="rgbd_camera_joint" type="fixed">
+			<origin xyz="0.05 0 0.1" rpy="0 0 0"/>
+			<parent link="front_mount"/>
+			<child link="rgbd_camera_frame"/>
+		</joint>
+		<link name="rgbd_camera_frame">
+			<visual>
+				<origin xyz="0 0 0" rpy="${PI/2} 0 ${PI/2}"/>
+				<geometry>
+					<mesh filename="file://$(find depth_d455)/meshes/d455.stl" scale="0.001 0.001 0.001"/>
+				</geometry>
+				<material name="aluminum">
+					<color rgba="0.5 0.5 0.5 1.0"/>
+				</material>
+			</visual>
+			<collision>
+				<origin xyz="0 0 0" rpy="0 0 0"/>
+				<geometry>
+					<box size="0.026 0.124 0.029"/>
+				</geometry>
+			</collision>
+			<inertial>
+				<origin xyz="0 0 0" rpy="0 0 0"/>
+				<mass value="0.12"/>
+				<inertia ixx="0.0001" ixy="0" ixz="0" iyy="0.0001" iyz="0" izz="0.0001"/>
+			</inertial>
+		</link>
 		<link name="rear_mount" />
 		<joint name="rear_mount_joint" type="fixed">
