Commit message: init drl for hunter se robot

File: ros2_ws/src/hunter_se_gazebo/urdf/mobile_robot/hunter_se.urdf.xacro (robot description, xacro)
@@ -1,5 +1,5 @@
 <?xml version="1.0"?>
 <!--
-  AgileX Hunter SE – main robot URDF macro (sensor-free).
+  AgileX Hunter SE – main robot URDF macro.
   Dimensions tuned toward the HUNTER SE V2.0.0 user manual:
     Wheelbase      : 0.5477 m
@@ -11,5 +11,5 @@
   Drive type: Ackermann steering (front-wheel steer, rear-wheel drive).
   Matches VehicleController.cs FrontWheelSteer + IRWD configuration.
-  Sensors: none. Add sensor xacro includes here when ready.
+  Sensors: Ouster OS1-64 + 2-D planar LiDAR.
   Visual meshes are stored in this package so the current simulation can stay
   self-contained.
@@ -30,6 +30,8 @@
     <xacro:property name="wheelbase"             value="${front_axle_x - rear_axle_x}"/>
     <xacro:property name="track"                 value="0.503404"/>
-    <!-- wheel-center Z relative to base_link (negative = below body center) -->
-    <xacro:property name="wheel_vertical_offset" value="-0.16713"/>
+    <!-- wheel-center Z relative to base_link (negative = below body center).
+         Raised by 3 mm so the chassis sits 3 mm lower while wheel contact
+         with the ground stays unchanged. -->
+    <xacro:property name="wheel_vertical_offset" value="-0.16413"/>
     <xacro:property name="wheel_radius" value="0.136"/>
     <xacro:property name="wheel_length" value="0.100"/>
@@ -39,7 +41,7 @@
     <link name="base_footprint"/>
     <joint name="base_footprint_to_base_link" type="fixed">
-      <!-- z = wheel_radius - wheel_vertical_offset = 0.136 - (-0.16713)
-           = 0.30313 m. Together with the imported visual mesh offset, this
-           yields about 817.55 x 644.0 x 303.63 mm at zero steering. -->
+      <!-- z = wheel_radius - wheel_vertical_offset = 0.136 - (-0.16413)
+           = 0.30013 m. Together with the imported visual mesh offset, this
+           yields about 817.55 x 644.0 x 300.63 mm at zero steering. -->
       <origin xyz="0 0 ${wheel_radius - wheel_vertical_offset}" rpy="0 0 0"/>
       <parent link="base_footprint"/>
@@ -94,4 +96,23 @@
       <child link="inertial_link"/>
     </joint>
+    <!-- ==================== 3-D OUSTER LIDAR ==================== -->
+    <!-- Placement derived from hunter_se_unity/:
+         Unity sensor origin = LIDAR mount (0, 0.6398543, -0.123163)
+         + Velodyne mount (0, -0.04, 0)
+         + Ouster child offset (0, 0.001310061, 0.03654947),
+         remapped to REP-103 axes. -->
+    <xacro:include filename="$(find ouster_description)/urdf/os1_64.urdf.xacro"/>
+    <xacro:os1_64 parent="mobile_robot_base"
+                  name="ouster"
+                  hz="10"
+                  samples="1024"
+                  min_range="0.5"
+                  max_range="100.0"
+                  min_angle_v="-21.2"
+                  max_angle_v="21.2"
+                  noise="0.01"
+                  topic="/hunter_se/pointcloud/points">
+      <origin xyz="-0.020851 0 0.430210" rpy="0 0 0"/>
+    </xacro:os1_64>
     <!-- ==================== WHEELS ==================== -->
     <xacro:include filename="$(find hunter_se_gazebo)/urdf/mobile_robot/hunter_se_wheel.xacro"/>
@@ -116,4 +137,37 @@
       wheel_mesh="${mesh_root}/re_right_link.STL"
       wheel_visual_rpy="-1.5708 0 0"/>
+    <!-- ==================== 2-D LIDAR ==================== -->
+    <!-- Mounted at robot center, 0.15 m above mobile_robot_base_link
+         (clears the 0.19 m body box whose top is at z≈0.103 m).
+         Frame: lidar_link (z-up, x-forward, matches REP 103). -->
+    <link name="lidar_link">
+      <visual>
+        <origin xyz="0 0 0" rpy="0 0 0"/>
+        <geometry>
+          <cylinder radius="0.04" length="0.04"/>
+        </geometry>
+        <material name="lidar_black">
+          <color rgba="0.1 0.1 0.1 1.0"/>
+        </material>
+      </visual>
+      <collision>
+        <origin xyz="0 0 0" rpy="0 0 0"/>
+        <geometry>
+          <cylinder radius="0.04" length="0.04"/>
+        </geometry>
+      </collision>
+      <inertial>
+        <mass value="0.2"/>
+        <origin xyz="0 0 0"/>
+        <inertia ixx="0.0001" ixy="0" ixz="0"
+                 iyy="0.0001" iyz="0"
+                 izz="0.0001"/>
+      </inertial>
+    </link>
+    <joint name="lidar_joint" type="fixed">
+      <origin xyz="0 0 0.15" rpy="0 0 0"/>
+      <parent link="mobile_robot_base_link"/>
+      <child link="lidar_link"/>
+    </joint>
     <!-- ==================== GAZEBO PLUGINS ==================== -->
     <xacro:if value="${load_gazebo}">

File: ros2_ws/src/hunter_se_gazebo/urdf/robot.urdf.xacro (robot description, xacro)
@@ -1,5 +1,5 @@
 <?xml version="1.0"?>
 <!--
-  Top-level xacro entry point for the Hunter SE robot (sensor-free).
+  Top-level xacro entry point for the Hunter SE robot.
   Args:
     load_gazebo : true (default) | false

File: ros2_ws/src/ouster_simulation/ouster_description/urdf/os1_64.urdf.xacro (robot description, xacro)
@@ -4,5 +4,5 @@
 <robot xmlns:xacro="http://ros.org/wiki/xacro" name="os1_64">
   <xacro:property name="PI" value="3.1415926535897931"/>
-  <xacro:macro name="os1_64" params="*origin parent:=base name:=os reduced:=true prefix:=/os1_cloud_node hz:=10 samples:=512 min_range:=0.8 max_range:=100 noise:=0.008 min_angle_v:=-16.6 max_angle_v:=16.6">
+  <xacro:macro name="os1_64" params="*origin parent:=base name:=os reduced:=true prefix:=/os1_cloud_node hz:=10 samples:=512 min_range:=0.8 max_range:=100 noise:=0.008 min_angle_v:=-16.6 max_angle_v:=16.6 topic:=/scout/pointcloud/points">
     <xacro:property name="file_visual" value="os1_64"/>
     <joint name="${name}_joint" type="fixed">
@@ -57,5 +57,5 @@
           <update_on_paused_sim>false</update_on_paused_sim>
           <!-- Match ros_gz_bridge mapping in your launch -->
-          <topic>/scout/pointcloud/points</topic>
+          <topic>${topic}</topic>
           <!-- frame_id in PointCloudPacked header -->
           <frame>${name}_lidar</frame>

Commit message: init first full system

File: ros2_ws/src/hunter_se_gazebo/urdf/mobile_robot/hunter_se.urdf.xacro (robot description, xacro)
@@ -7,9 +7,9 @@
     Wheel radius   : 0.136 m
     Wheel length   : 0.100 m  (tyre width)
-    Body (approx)  : 820 × 440 × 190 mm  (collision box, excluding wheel protrusion)
+    Body (approx)  : 760 × 400 × 140 mm  (collision box, front face aligned to wheel front)
     Total mass     : 42.0 kg
   Drive type: Ackermann steering (front-wheel steer, rear-wheel drive).
   Matches VehicleController.cs FrontWheelSteer + IRWD configuration.
-  Sensors: Ouster OS1-64 + 2-D planar LiDAR.
+  Sensors: Ouster OS1-64 (3-D PointCloud2 → /scan via pointcloud_to_laserscan).
   Visual meshes are stored in this package so the current simulation can stay
   self-contained.
@@ -18,8 +18,18 @@
   <xacro:macro name="hunter_se" params="load_gazebo">
     <!-- ==================== DIMENSIONS ==================== -->
-    <!-- Body collision box (excluding wheel protrusion) -->
-    <xacro:property name="base_x_size" value="0.820"/>
-    <xacro:property name="base_y_size" value="0.440"/>
-    <xacro:property name="base_z_size" value="0.190"/>
+    <!-- Body collision box.
+         Keep the chassis collision slightly inside the visual mesh in Y/Z,
+         while aligning the front face with the front wheel collision envelope:
+           front wheel foremost x = front_axle_x + wheel_radius = 0.475638 m
+         With a shorter body box, shift the collision box forward so its front
+         face lands at that x coordinate. -->
+    <xacro:property name="base_x_size" value="0.760"/>
+    <xacro:property name="base_y_size" value="0.400"/>
+    <xacro:property name="base_z_size" value="0.140"/>
+    <xacro:property name="base_collision_x_offset" value="${front_axle_x + wheel_radius - base_x_size/2}"/>
+    <!-- Place the bottom face of the main body collision box at the wheel
+         centre height so the chassis collision starts above the wheel-contact
+         band instead of extending unrealistically low. -->
+    <xacro:property name="base_collision_z_center" value="${wheel_vertical_offset + base_z_size/2}"/>
     <!-- Ackermann kinematics / mesh placement.
          Axles are not perfectly symmetric about the base origin because the
@@ -31,7 +41,7 @@
     <xacro:property name="track"                 value="0.503404"/>
     <!-- wheel-center Z relative to base_link (negative = below body center).
-         Raised by 3 mm so the chassis sits 3 mm lower while wheel contact
+         Raised by 8 mm total so the chassis sits 8 mm lower while wheel contact
          with the ground stays unchanged. -->
-    <xacro:property name="wheel_vertical_offset" value="-0.16413"/>
+    <xacro:property name="wheel_vertical_offset" value="-0.15913"/>
     <xacro:property name="wheel_radius" value="0.136"/>
     <xacro:property name="wheel_length" value="0.100"/>
@@ -41,7 +51,7 @@
     <link name="base_footprint"/>
     <joint name="base_footprint_to_base_link" type="fixed">
-      <!-- z = wheel_radius - wheel_vertical_offset = 0.136 - (-0.16413)
-           = 0.30013 m. Together with the imported visual mesh offset, this
-           yields about 817.55 x 644.0 x 300.63 mm at zero steering. -->
+      <!-- z = wheel_radius - wheel_vertical_offset = 0.136 - (-0.15913)
+           = 0.29513 m. Together with the imported visual mesh offset, this
+           yields about 817.55 x 644.0 x 295.63 mm at zero steering. -->
       <origin xyz="0 0 ${wheel_radius - wheel_vertical_offset}" rpy="0 0 0"/>
       <parent link="base_footprint"/>
@@ -65,7 +75,7 @@
         </material>
       </visual>
-      <!-- Two collision boxes: main body + raised centre rail -->
+      <!-- Two collision boxes: main body + narrowed raised centre rail -->
       <collision>
-        <origin xyz="0 0 0.008" rpy="0 0 0"/>
+        <origin xyz="${base_collision_x_offset} 0 ${base_collision_z_center}" rpy="0 0 0"/>
         <geometry>
           <box size="${base_x_size} ${base_y_size} ${base_z_size}"/>
@@ -73,7 +83,7 @@
       </collision>
       <collision>
-        <origin xyz="0 0 ${base_z_size/6}" rpy="0 0 0"/>
+        <origin xyz="${base_collision_x_offset} 0 ${base_collision_z_center + base_z_size/6}" rpy="0 0 0"/>
         <geometry>
-          <box size="${base_x_size/5} ${base_y_size*1.5} ${base_z_size/3}"/>
+          <box size="${base_x_size/4} ${base_y_size*0.5} ${base_z_size/3}"/>
         </geometry>
       </collision>
@@ -96,5 +106,5 @@
       <child link="inertial_link"/>
     </joint>
-    <!-- ==================== 3-D OUSTER LIDAR ==================== -->
+    <!-- ==================== 3-D OUSTER OS1-128 LIDAR ==================== -->
     <!-- Placement derived from hunter_se_unity/:
          Unity sensor origin = LIDAR mount (0, 0.6398543, -0.123163)
@@ -105,13 +115,14 @@
     <xacro:os1_64 parent="mobile_robot_base"
                   name="ouster"
+                  channels="128"
                   hz="10"
-                  samples="1024"
-                  min_range="0.5"
-                  max_range="100.0"
-                  min_angle_v="-21.2"
-                  max_angle_v="21.2"
+                  samples="2048"
+                  min_range="0.3"
+                  max_range="120.0"
+                  min_angle_v="-22.5"
+                  max_angle_v="22.5"
                   noise="0.01"
                   topic="/hunter_se/pointcloud/points">
-      <origin xyz="-0.020851 0 0.430210" rpy="0 0 0"/>
+      <origin xyz="0 0 0.304870" rpy="0 0 0"/>
     </xacro:os1_64>
     <!-- ==================== WHEELS ==================== -->
@@ -137,37 +148,4 @@
       wheel_mesh="${mesh_root}/re_right_link.STL"
       wheel_visual_rpy="-1.5708 0 0"/>
-    <!-- ==================== 2-D LIDAR ==================== -->
-    <!-- Mounted at robot center, 0.15 m above mobile_robot_base_link
-         (clears the 0.19 m body box whose top is at z≈0.103 m).
-         Frame: lidar_link (z-up, x-forward, matches REP 103). -->
-    <link name="lidar_link">
-      <visual>
-        <origin xyz="0 0 0" rpy="0 0 0"/>
-        <geometry>
-          <cylinder radius="0.04" length="0.04"/>
-        </geometry>
-        <material name="lidar_black">
-          <color rgba="0.1 0.1 0.1 1.0"/>
-        </material>
-      </visual>
-      <collision>
-        <origin xyz="0 0 0" rpy="0 0 0"/>
-        <geometry>
-          <cylinder radius="0.04" length="0.04"/>
-        </geometry>
-      </collision>
-      <inertial>
-        <mass value="0.2"/>
-        <origin xyz="0 0 0"/>
-        <inertia ixx="0.0001" ixy="0" ixz="0"
-                 iyy="0.0001" iyz="0"
-                 izz="0.0001"/>
-      </inertial>
-    </link>
-    <joint name="lidar_joint" type="fixed">
-      <origin xyz="0 0 0.15" rpy="0 0 0"/>
-      <parent link="mobile_robot_base_link"/>
-      <child link="lidar_link"/>
-    </joint>
     <!-- ==================== GAZEBO PLUGINS ==================== -->
     <xacro:if value="${load_gazebo}">

File: ros2_ws/src/ouster_simulation/ouster_description/urdf/os1_64.urdf.xacro (robot description, xacro)
@@ -2,7 +2,8 @@
 <!-- Modified from the work of Wil Selby (https://github.com/wilselby/ouster_example/blob/master/ouster_description/urdf/OS1-64.urdf.xacro) -->
 <!-- Updated for Gazebo Ignition (Gazebo Sim) compatibility -->
+<!-- Configurable OS1 family macro; Hunter SE overrides this to OS1-128 settings. -->
 <robot xmlns:xacro="http://ros.org/wiki/xacro" name="os1_64">
   <xacro:property name="PI" value="3.1415926535897931"/>
-  <xacro:macro name="os1_64" params="*origin parent:=base name:=os reduced:=true prefix:=/os1_cloud_node hz:=10 samples:=512 min_range:=0.8 max_range:=100 noise:=0.008 min_angle_v:=-16.6 max_angle_v:=16.6 topic:=/scout/pointcloud/points">
+  <xacro:macro name="os1_64" params="*origin parent:=base name:=os reduced:=true prefix:=/os1_cloud_node hz:=10 channels:=64 samples:=1024 min_range:=0.5 max_range:=100 noise:=0.008 min_angle_v:=-21.2 max_angle_v:=21.2 topic:=/scout/pointcloud/points">
     <xacro:property name="file_visual" value="os1_64"/>
     <joint name="${name}_joint" type="fixed">
@@ -62,21 +63,20 @@
           <!-- Use uniform pattern with explicit vertical FOV -->
           <!-- NOTE: pattern_preset "OS1 64" has 0° vertical FOV (bug), using pattern_uniform instead -->
-          <!-- Ouster OS1-64: 64 channels, 1024 horizontal samples, ±16.6° vertical FOV -->
-          <!-- Angles in radians: 16.6° = 0.2897 rad, 180° = 3.14159 rad -->
+          <!-- All angle parameters here are passed in degrees and converted to radians. -->
           <pattern_uniform>
             <horizontal>
-              <samples>1024</samples>
+              <samples>${samples}</samples>
               <min_angle>-3.14159</min_angle>
               <max_angle>3.14159</max_angle>
             </horizontal>
             <vertical>
-              <samples>64</samples>
-              <min_angle>-0.2897</min_angle>
-              <max_angle>0.2897</max_angle>
+              <samples>${channels}</samples>
+              <min_angle>${min_angle_v*PI/180.0}</min_angle>
+              <max_angle>${max_angle_v*PI/180.0}</max_angle>
             </vertical>
           </pattern_uniform>
           <!-- Channel configuration for ring ID and timestamp support -->
-          <channels>64</channels>
-          <horizontal_samples>1024</horizontal_samples>
+          <channels>${channels}</channels>
+          <horizontal_samples>${samples}</horizontal_samples>
           <noise>
             <mean>0.0</mean>

Commit message: fix some errors

File: ros2_ws/src/hunter_se_gazebo/urdf/mobile_robot/hunter_se.urdf.xacro (robot description, xacro)
@@ -124,5 +124,5 @@
                   noise="0.01"
                   topic="/hunter_se/pointcloud/points">
-      <origin xyz="0 0 0.304870" rpy="0 0 0"/>
+      <origin xyz="0 0 0.204870" rpy="0 0 0"/>
     </xacro:os1_64>
     <!-- ==================== WHEELS ==================== -->

Commit message: apply dynamic obstacles in drl_arena

File: ros2_ws/src/hunter_se_gazebo/urdf/mobile_robot/hunter_se.urdf.xacro (robot description, xacro)
@@ -11,5 +11,5 @@
   Drive type: Ackermann steering (front-wheel steer, rear-wheel drive).
   Matches VehicleController.cs FrontWheelSteer + IRWD configuration.
-  Sensors: Ouster OS1-64 (3-D PointCloud2 → /scan via pointcloud_to_laserscan).
+  Sensors: Ouster OS1-128 (3-D PointCloud2 → /scan via pointcloud_to_laserscan).
   Visual meshes are stored in this package so the current simulation can stay
   self-contained.
@@ -76,5 +76,5 @@
       </visual>
       <!-- Two collision boxes: main body + narrowed raised centre rail -->
-      <collision>
+      <collision name="chassis_collision">
         <origin xyz="${base_collision_x_offset} 0 ${base_collision_z_center}" rpy="0 0 0"/>
         <geometry>
@@ -82,5 +82,5 @@
         </geometry>
       </collision>
-      <collision>
+      <collision name="center_rail_collision">
         <origin xyz="${base_collision_x_offset} 0 ${base_collision_z_center + base_z_size/6}" rpy="0 0 0"/>
         <geometry>
